File: 00-proyecto-02/grupo-01/piezo-02-v03/piezo-02-v03.kicad_sch (KiCad schematic)
At the start: 27 parts, among them J1 TTS, J2 TTS, Q1 PN2222A, U1 LM324

Commit message: agregar PWR_FLAG y borrar V_BUS
Connections:
- net VBUS: no longer names the net of C4.1, C5.1, R4.1, U1.13 (-), U1.14, U1.5 (+)
